Commit message: versao atualizada - modelo urdf funcional - MoveIt versao inicial instalada .

File: RosTests/catkin_ws/src/tangs5dof/urdf/robot.urdf (robot description, URDF)
Before this commit: robot onshape, 6 links, 5 joints
Links:
- removed link arm1
- removed link arm2
- removed link arm3
- removed link base
- removed link part_1
- added link link_arm, mass 0.079963772883510669809; collision mesh filename=package://tangs5dof/urdf/link_arm.stl; visual mesh filename=package://tangs5dof/urdf/link_arm.stl
- added link link_base, mass 0.12002083594684367918; collision mesh filename=package://tangs5dof/urdf/link_base.stl; visual mesh filename=package://tangs5dof/urdf/link_base.stl
- added link link_body, mass 0.085013969989408674777; collision mesh filename=package://tangs5dof/urdf/link_body.stl; visual mesh filename=package://tangs5dof/urdf/link_body.stl
- added link link_forearm, mass 0.052819407015602941324; collision mesh filename=package://tangs5dof/urdf/link_forearm.stl; visual mesh filename=package://tangs5dof/urdf/link_forearm.stl
- added link link_hand, mass 0.018279517977360375258; collision mesh filename=package://tangs5dof/urdf/link_hand.stl; visual mesh filename=package://tangs5dof/urdf/link_hand.stl
- added link link_palm, mass 0.020500595775101038837; collision mesh filename=package://tangs5dof/urdf/link_palm.stl; visual mesh filename=package://tangs5dof/urdf/link_palm.stl
Joints:
- removed joint end_effector
- added joint wrist_pitch: type revolute, parent link_hand, child link_palm, origin xyz=0.0049813961386296901068 -0.014010243159726681883 -0.027996103280433365379 rpy=-1.570796326794896558 -0.038080793091696346631 -5.4995910972554887091e-15, axis 0 0 1, limit lower=-1.570796326794896558 upper=1.570796326794896558 effort=1 velocity=20
- added joint wrist_yaw: type revolute, parent link_forearm, child link_hand, origin xyz=-0.0053082245392911675541 -0.089748321005440834242 -0.0075144749285244276382 rpy=-1.570796326794896558 -0.26234740040539716865 7.9319393344061070401e-15, axis 0 0 1, limit lower=-1.570796326794896558 upper=1.570796326794896558 effort=1 velocity=20
- joint dummy_joint: child arm3 -> link_base
- joint elbow: child part_1 -> link_forearm; limit lower=0 upper=3.141592653589793116 effort=1 velocity=20 -> lower=-3.141592653589793116 upper=2.0943951023931952626 effort=1 velocity=20; origin xyz=0.11998739918318486464 -2.123187930913594812e-06 -3.4694469519536141888e-18 rpy=-3.3269375668139454439e-15 2.1475876632594051176e-15 1.0742051321332899416 -> xyz=-0.11998739918318489239 -2.1231879309170642589e-06 1.7347234759768070944e-18 rpy=3.141592653589793116 -7.8822160764989523078e-16 0.60886401637823828192; parent arm1 -> link_arm
- joint shoulder: child base -> link_arm; origin xyz=-0.013965289960663616886 -0.040301559464014063972 0.0040000001899898052216 rpy=-1.570796326794896558 -0.012551015857183739355 -4.1254338333079384561e-23 -> xyz=-0.0040000001899898043542 0.013965289960663616886 0.040301559464014063972 rpy=1.5707963267953313213 1.5702417558227264038 -1.570796326798316267; parent part_1 -> link_body
- joint waist: child arm1 -> link_body; limit lower=0 upper=4.712388980384689674 effort=1 velocity=20 -> lower=-1.570796326794896558 upper=1.570796326794896558 effort=1 velocity=20; origin xyz=0.0053082245392913340876 0.0075144749285244241688 -0.089748321005440917508 rpy=1.570796326794896558 -0.56539704268284429745 3.1415926535897891192 -> xyz=5.0306980803327405738e-17 1.3114530717629603727e-18 0.056000001728534705425 rpy=2.0816681711721669356e-15 4.5796699765786533862e-16 1.5455769190268391355; parent arm2 -> link_base

Commit message: Ajustes nos arquivos - visualização e simulação ok

File: RosTests/catkin_ws/src/tangs5dof/urdf/robot.urdf (robot description, URDF)
Before this commit: robot onshape, 7 links, 6 joints
Joints:
- joint elbow: limit lower=-3.141592653589793116 upper=2.0943951023931952626 effort=1 velocity=20 -> lower=-3.141592653589793116 upper=2.0943951023931952626 effort=1 velocity=0.5
- joint shoulder: limit lower=-1.570796326794896558 upper=1.570796326794896558 effort=1 velocity=20 -> lower=-1.570796326794896558 upper=1.570796326794896558 effort=2 velocity=1.0
- joint waist: limit lower=-1.570796326794896558 upper=1.570796326794896558 effort=1 velocity=20 -> lower=-1.570796326794896558 upper=1.570796326794896558 effort=0.1 velocity=0.5
- joint wrist_pitch: limit lower=-1.570796326794896558 upper=1.570796326794896558 effort=1 velocity=20 -> lower=-1.570796326794896558 upper=1.570796326794896558 effort=1 velocity=0.5
- joint wrist_yaw: limit lower=-1.570796326794896558 upper=1.570796326794896558 effort=1 velocity=20 -> lower=-1.570796326794896558 upper=1.570796326794896558 effort=2 velocity=0.5

File: RosTests/catkin_ws/src/tangs5dof/urdf/robot_onecontroller.urdf (robot description, URDF)
Before this commit: robot onshape, 7 links, 6 joints
Joints:
- joint waist: limit lower=-1.570796326794896558 upper=1.570796326794896558 effort=1 velocity=20 -> lower=-1.570796326794896558 upper=1.570796326794896558 effort=0.1 velocity=0.5
