Commit message: Versão do projeto com a pasta de simulação e Controle do roomba com o rpi.

File: rosurdf_tutorial/simple_robot_ws/src/robot_articulated/description/robot.urdf.xacro (robot description, xacro)
@@ -2,3 +2,4 @@
 <robot xmlns:xacro="http://www.ros.org/wiki/xacro" name="firefighter">
     <xacro:include filename="$(find robot_articulated)/description/robot_core.xacro"/>
+    <!-- <xacro:include filename="$(find robot_articulated)/description/gazebo_control.xacro"/> -->
 </robot>

File: rosurdf_tutorial/simple_robot_ws/src/robot_articulated/description/robot_core.xacro (robot description, xacro)
@@ -1,4 +1,4 @@
 <?xml version="1.0"?>
-<robot xmlns:xacro="http://www.ros.org/wiki/xacro">
+<robot xmlns:xacro="http://www.ros.org/wiki/xacro" >
     <xacro:include filename="inertial_macros.xacro"/>
     <material name="white">
@@ -14,8 +14,8 @@
         <color rgba="0 0 0 1"/>
     </material>
-    <!-- BASE LINK -->
-    <link name="base_link">
-    </link>
-    <!-- CHASSIS LINK -->
+   <!-- BASE LINK -->
+   <link name="base_link">
+   </link>
+   <!-- Chassis -->
     <joint name="chassis_joint" type="fixed">
         <parent link="base_link"/>
@@ -41,35 +41,15 @@
         </xacro:inertial_cylinder>
     </link>
+    <gazebo reference="chassis">
+        <material>Gazebo/White</material>
+    </gazebo>
     <!-- LEFT WHEEL Link -->
-    <joint name = "left_wheel_joint" type = "continuous">
-        <parent link="base_link"/>
-        <child link="left_wheel"/>
-        <origin xyz="0.0 0.10 0.0" rpy="-${pi/2} 0.0 0.0"/>
-        <axis xyz="0.0 0.0 1.0"/>
-    </joint>
-    <link name = "left_wheel">
-        <visual>
-            <geometry>
-                <cylinder radius="0.03" length="0.02"/>
-            </geometry>
-            <material name = "blue"/>
-        </visual>
-        <collision>
-            <geometry>
-                <cylinder radius="0.03" length="0.02"/>
-            </geometry>
-        </collision>
-        <xacro:inertial_cylinder mass="0.1" length="0.02" radius="0.03">
-            <origin xyz="0 0 0" rpy="0 0 0"/>
-        </xacro:inertial_cylinder>
-    </link>
-        <!-- RIGHT WHEEL Link -->
-        <joint name = "right_wheel_joint" type = "continuous">
-            <parent link="base_link"/>
-            <child link="right_wheel"/>
-            <origin xyz="0.0 -0.10 0.0" rpy="${pi/2} 0.0 0.0"/>
-            <axis xyz="0.0 0.0 -1.0"/>
-        </joint>
-        <link name = "right_wheel">
+                <joint name = "left_wheel_joint" type = "continuous">
+                    <parent link="base_link"/>
+                    <child link="left_wheel"/>
+                    <origin xyz="0.0 0.10 0.0" rpy="-${pi/2} 0.0 0.0"/>
+                    <axis xyz="0.0 0.0 1.0"/>
+                </joint>
+        <link name = "left_wheel">
             <visual>
                 <geometry>
@@ -87,25 +67,59 @@
             </xacro:inertial_cylinder>
         </link>
-        <!-- Caster Wheel link -->
-        <joint name = "caster_wheel_joint" type = "fixed">
-            <parent link="base_link"/>
-            <child link="caster_wheel"/>
-            <origin xyz="0.12 0.0 0.0" />
-        </joint>
-        <link name = "caster_wheel">
-            <visual>
-                <geometry>
-                    <sphere radius="0.03"/>
-                </geometry>
-                <material name = "black"/>
-            </visual>
-            <collision>
-                <geometry>
-                    <sphere radius="0.03"/>
-                </geometry>
-            </collision>
-            <xacro:inertial_sphere mass="0.1" radius="0.03">
-                <origin xyz="0 0 0" rpy="0 0 0"/>
-            </xacro:inertial_sphere>
-        </link>
+        <gazebo reference="left_wheel">
+            <material>Gazebo/Blue</material>
+        </gazebo>
+            <!-- RIGHT WHEEL Link -->
+            <joint name = "right_wheel_joint" type = "continuous">
+                <parent link="base_link"/>
+                <child link="right_wheel"/>
+                <origin xyz="0.0 -0.10 0.0" rpy="${pi/2} 0.0 0.0"/>
+                <axis xyz="0.0 0.0 -1.0"/>
+            </joint>
+            <link name = "right_wheel">
+                <visual>
+                    <geometry>
+                        <cylinder radius="0.03" length="0.02"/>
+                    </geometry>
+                    <material name = "blue"/>
+                </visual>
+                <collision>
+                    <geometry>
+                        <cylinder radius="0.03" length="0.02"/>
+                    </geometry>
+                </collision>
+                <xacro:inertial_cylinder mass="0.1" length="0.02" radius="0.03">
+                    <origin xyz="0 0 0" rpy="0 0 0"/>
+                </xacro:inertial_cylinder>
+            </link>
+            <gazebo reference="right_wheel">
+                <material>Gazebo/Blue</material>
+            </gazebo>
+            <!-- Caster Wheel link -->
+            <joint name = "caster_wheel_joint" type = "fixed">
+                <parent link="base_link"/>
+                <child link="caster_wheel"/>
+                <origin xyz="0.12 0.0 0.0" />
+            </joint>
+            <link name = "caster_wheel">
+                <visual>
+                    <geometry>
+                        <sphere radius="0.03"/>
+                    </geometry>
+                    <material name = "black"/>
+                </visual>
+                <collision>
+                    <geometry>
+                        <sphere radius="0.03"/>
+                    </geometry>
+                </collision>
+                <xacro:inertial_sphere mass="0.1" radius="0.03">
+                    <origin xyz="0 0 0" rpy="0 0 0"/>
+                </xacro:inertial_sphere>
+            </link>
+            <gazebo reference="caster_wheel">
+                <material>Gazebo/Black</material>
+                <mu1 value="0.001"/>
+                <mu2 value="0.001"/>
+            </gazebo>
 </robot>
